File: sd/v1.4/Fubarino_SD_v14t.sch (EAGLE design)
At the start: 35 parts, among them IC1 PIC32MX440F256H-80I/PT, J8 UX60A-MB-5ST, Q1 8.000MHz, Q2 32.768 KHz

Commit message: Adjusted pads/holes for SD, buttons, and lock headers: cobra18t <https://github.com/cobra18t>
Parts:
- JP1, JP2, JP3, JP4: device SparkFun:M14LOCK -> TEF_made3:M14LOCK
- PROGRAM, RESET: device SparkFun02-20-08:TAC_SWITCHSND -> TEF_made3:TAC_SWITCHSMD
Changed lines of the file:
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@@
 <part name="R9" library="SparkFun" deviceset="RESISTOR" device="0603-RES" value="10K"/>
 <part name="R3" library="SparkFun" deviceset="RESISTOR" device="0603-RES" value="10K"/>
-<part name="PROGRAM" library="SparkFun02-20-08" deviceset="TAC_SWITCH" device="SND" value="PTS525SM10SMTR LFS"/>
+<part name="PROGRAM" library="TEF_made3" deviceset="TAC_SWITCH" device="SMD" value="PTS525SM10SMTR LFS"/>
 <part name="P+16" library="SparkFun02-20-08" deviceset="3.3V" device=""/>
-<part name="RESET" library="SparkFun02-20-08" deviceset="TAC_SWITCH" device="SND" value="PTS525SM10SMTR LFS"/>
+<part name="RESET" library="TEF_made3" deviceset="TAC_SWITCH" device="SMD" value="PTS525SM10SMTR LFS"/>
 <part name="R10" library="SparkFun" deviceset="RESISTOR" device="0603-RES" value="10K"/>
 <part name="R11" library="SparkFun" deviceset="RESISTOR" device="0603-RES" value="330"/>
@@
 <part name="GND13" library="SparkFun02-20-08" deviceset="GND" device=""/>
 <part name="IC3" library="SparkFun" deviceset="V_REG_LM1117" device="SOT223"/>
-<part name="JP1" library="SparkFun" deviceset="M14" device="LOCK"/>
-<part name="JP2" library="SparkFun" deviceset="M14" device="LOCK"/>
+<part name="JP1" library="TEF_made3" deviceset="M14" device="LOCK"/>
+<part name="JP2" library="TEF_made3" deviceset="M14" device="LOCK"/>
 <part name="U$2" library="TEF_made3" deviceset="SDCARD" device="MICROSD1"/>
 <part name="SJ1" library="SparkFun" deviceset="SOLDERJUMPER" device="TRACE"/>
-<part name="JP3" library="SparkFun" deviceset="M14" device="LOCK"/>
-<part name="JP4" library="SparkFun" deviceset="M14" device="LOCK"/>
+<part name="JP3" library="TEF_made3" deviceset="M14" device="LOCK"/>
+<part name="JP4" library="TEF_made3" deviceset="M14" device="LOCK"/>
 <part name="Q1" library="TEF_made3" deviceset="METRIC_XTAL" device="6035_METRIC" value="8.000MHz"/>
 <part name="D1" library="diode" deviceset="DIODE-" device="SOD123"/>
